File: source/geheimbadge-controller/geheimbadge-controller.kicad_pcb (KiCad board)
At the start: 2 copper layers, 75.9 x 74.5 mm, 1 part, among them J1 SAOv2

Commit message: finalized controller design
Parts:
- added BT1: Conn_01x02_MountingPin, Connector_JST:JST_PH_S2B-PH-SM4-TB_1x02-1MP_P2.00mm_Horizontal, F.Cu at (113.5, 97.0)
- added C1: 10u, Capacitor_SMD:C_0805_2012Metric, F.Cu at (121.0, 90.0)
- added C10: 100n, Capacitor_SMD:C_0603_1608Metric, F.Cu at (108.0, 146.0)
- added C11: 10u, Capacitor_SMD:C_0805_2012Metric, F.Cu at (110.0, 146.0)
- added C2: 100n, Capacitor_SMD:C_0603_1608Metric, F.Cu at (89.5, 92.0)
- added C3: 100n, Capacitor_SMD:C_0603_1608Metric, F.Cu at (75.0, 97.0)
- added C4: 10u, Capacitor_SMD:C_0805_2012Metric, F.Cu at (121.0, 97.5)
- added C5: 10u, Capacitor_SMD:C_0805_2012Metric, F.Cu at (85.5, 99.5)
- added C6: 10u, Capacitor_SMD:C_0805_2012Metric, F.Cu at (128.0, 115.0)
- added C7: 10u, Capacitor_SMD:C_0805_2012Metric, F.Cu at (135.0, 115.0)
- added C8: 10u, Capacitor_SMD:C_0805_2012Metric, F.Cu at (87.5, 120.5)
- added C9: 10u, Capacitor_SMD:C_0805_2012Metric, F.Cu at (91.0, 120.5)
- added D1: LED, LED_SMD:LED_0603_1608Metric, F.Cu at (114.0, 90.5)
- added D2: 1N4148WS, Diode_SMD:D_SOD-323, F.Cu at (125.0, 92.5)
- added D3: 1N4148WS, Diode_SMD:D_SOD-323, F.Cu at (123.5, 102.5)
- added J2: Conn_01x06, Connector_PinSocket_2.54mm:PinSocket_1x06_P2.54mm_Horizontal, F.Cu at (82.0, 124.0)
- added J3: SAOv2, Connector_PinSocket_2.54mm:PinSocket_2x03_P2.54mm_Vertical, F.Cu at (97.5, 124.7)
- added J4: Conn_01x06, Connector_PinSocket_2.54mm:PinSocket_1x06_P2.54mm_Horizontal, F.Cu at (109.0, 133.0)
- added JP1: Pmod_voltage, Jumper:SolderJumper-3_P1.3mm_Bridged12_RoundedPad1.0x1.5mm, B.Cu at (115.5, 121.5)
- added L1: 2.2uH, Inductor_SMD:L_1008_2520Metric, F.Cu at (129.5, 118.5)
- added L2: 2.2uH, Inductor_SMD:L_1008_2520Metric, F.Cu at (87.5, 123.5)
- added Q1: AO3400A, Package_TO_SOT_SMD:SOT-23, F.Cu at (126.5, 95.5)
- added Q2: MMDT3906, Package_TO_SOT_SMD:SOT-363_SC-70-6, F.Cu at (91.5, 98.5)
- added Q3: AO3401A, Package_TO_SOT_SMD:SOT-23, F.Cu at (95.5, 98.5)
- added Q4: AO3401A, Package_TO_SOT_SMD:SOT-23, F.Cu at (126.5, 99.5)
- added Q5: MMDT3906, Package_TO_SOT_SMD:SOT-363_SC-70-6, F.Cu at (131.5, 104.0)
- added Q6: AO3401A, Package_TO_SOT_SMD:SOT-23, F.Cu at (131.5, 108.0)
- added R1: 10k, Resistor_SMD:R_0603_1608Metric, F.Cu at (116.0, 90.5)
- added R10: 10, Resistor_SMD:R_0603_1608Metric, F.Cu at (79.5, 99.5)
- added R11: 180k, Resistor_SMD:R_0603_1608Metric, F.Cu at (123.5, 99.5)
- added R12: 10, Resistor_SMD:R_0603_1608Metric, F.Cu at (79.5, 101.5)
- added R13: 180k, Resistor_SMD:R_0603_1608Metric, F.Cu at (91.5, 101.5)
- added R14: 820k, Resistor_SMD:R_0603_1608Metric, F.Cu at (95.5, 101.5)
- added R15: 180k, Resistor_SMD:R_0603_1608Metric, F.Cu at (128.5, 104.0)
- added R16: 820k, Resistor_SMD:R_0603_1608Metric, F.Cu at (128.5, 108.0)
- added R17: 820k, Resistor_SMD:R_0603_1608Metric, F.Cu at (131.5, 111.0)
- added R18: 180k, Resistor_SMD:R_0603_1608Metric, F.Cu at (131.5, 112.5)
- added R19: 10k, Resistor_SMD:R_0603_1608Metric, F.Cu at (133.0, 117.5)
- added R2: 1k, Resistor_SMD:R_0603_1608Metric, F.Cu at (118.0, 90.5)
- added R20: 10, Resistor_SMD:R_0603_1608Metric, F.Cu at (108.5, 124.5)
- added R21: 10, Resistor_SMD:R_0603_1608Metric, F.Cu at (110.5, 124.5)
- added R22: 10k, Resistor_SMD:R_0603_1608Metric, F.Cu at (91.0, 126.0)
- added R23: 10k, Resistor_SMD:R_0603_1608Metric, F.Cu at (94.5, 131.5)
- added R24: 10k, Resistor_SMD:R_0603_1608Metric, F.Cu at (94.5, 134.5)
- added R25: 10, Resistor_SMD:R_0603_1608Metric, F.Cu at (91.5, 142.5)
- added R26: 10, Resistor_SMD:R_0603_1608Metric, F.Cu at (91.5, 144.0)
- added R3: 10k, Resistor_SMD:R_0603_1608Metric, F.Cu at (75.5, 92.0)
- added R4: 5.1k, Resistor_SMD:R_0603_1608Metric, F.Cu at (75.5, 93.5)
- added R5: 5.1k, Resistor_SMD:R_0603_1608Metric, F.Cu at (89.5, 93.5)
- added R6: 100k, Resistor_SMD:R_0603_1608Metric, F.Cu at (129.5, 95.5)
- added R7: 820k, Resistor_SMD:R_0603_1608Metric, F.Cu at (131.0, 95.5)
- added R8: 10k, Resistor_SMD:R_0603_1608Metric, F.Cu at (129.5, 98.5)
- added R9: 180k, Resistor_SMD:R_0603_1608Metric, F.Cu at (131.0, 98.5)
- added SW1: PWR, Button_Switch_SMD:SW_Push_1P1T_XKB_TS-1187A, B.Cu at (117.5, 92.5)
- added SW2: BOOT, Button_Switch_SMD:SW_Push_1P1T_XKB_TS-1187A, B.Cu at (89.5, 102.0)
- added SW3: RESET, Button_Switch_SMD:SW_Push_1P1T_XKB_TS-1187A, B.Cu at (75.5, 102.0)
- added TP1: TestPoint, TestPoint:TestPoint_Pad_D1.0mm, B.Cu at (84.0, 93.0)
- added TP10: TestPoint, TestPoint:TestPoint_Pad_D1.0mm, B.Cu at (80.5, 104.0)
- added TP11: TestPoint, TestPoint:TestPoint_Pad_D1.0mm, B.Cu at (136.0, 109.0)
- added TP12: TestPoint, TestPoint:TestPoint_Pad_D1.0mm, B.Cu at (133.5, 119.5)
- added TP13: TestPoint, TestPoint:TestPoint_Pad_D1.0mm, B.Cu at (119.0, 120.5)
- added TP14: TestPoint, TestPoint:TestPoint_Pad_D1.0mm, B.Cu at (112.0, 120.5)
- added TP15: TestPoint, TestPoint:TestPoint_Pad_D1.0mm, B.Cu at (94.0, 127.0)
- added TP2: TestPoint, TestPoint:TestPoint_Pad_D1.0mm, B.Cu at (81.0, 93.0)
- added TP3: TestPoint, TestPoint:TestPoint_Pad_D1.0mm, B.Cu at (86.0, 94.0)
- added TP4: TestPoint, TestPoint:TestPoint_Pad_D1.0mm, B.Cu at (79.0, 94.0)
- added TP5: TestPoint, TestPoint:TestPoint_Pad_D1.0mm, B.Cu at (117.0, 97.0)
- added TP6: TestPoint, TestPoint:TestPoint_Pad_D1.0mm, B.Cu at (134.0, 98.0)
- added TP7: TestPoint, TestPoint:TestPoint_Pad_D1.0mm, B.Cu at (134.0, 100.5)
- added TP8: TestPoint, TestPoint:TestPoint_Pad_D1.0mm, B.Cu at (121.0, 101.0)
- added TP9: TestPoint, TestPoint:TestPoint_Pad_D1.0mm, B.Cu at (84.5, 104.0)
- added U1: XC5011, Package_TO_SOT_SMD:TSOT-23-5, F.Cu at (121.0, 93.5)
- added U2: USBLC6-2SC6, Package_TO_SOT_SMD:SOT-23-6, F.Cu at (75.0, 100.5)
- added U3: TLV62568DBVR, Package_TO_SOT_SMD:SOT-23-5, F.Cu at (131.5, 115.0)
- added U4: XT1861B502SR-G, Package_TO_SOT_SMD:SOT-23-5, F.Cu at (91.0, 123.5)
- added U5: ESP32-C3-MINI-1-N4, ESP32-C3-MINI:WIFIM-SMD_ESP32-C3-MINI-1, F.Cu at (100.0, 143.0)
- J1: value SAOv2 -> USB_C_Receptacle_USB2.0; footprint Connector_PinSocket_2.54mm:PinSocket_2x03_P2.54mm_Vertical -> Connector_USB:USB_C_Receptacle_HRO_TYPE-C-31-M-12; moved to F.Cu
- moved J1 58.2 mm to (82.5, 93.0), turned to 180 degrees
Routing:
- net +3V3: track 0.00 -> 111.5 mm, vias 0 -> 5
- net +VDC: track 0.00 -> 102.0 mm, vias 0 -> 1
- net VBUS: track 0.00 -> 90.0 mm, vias 0 -> 3
- net /RESET: track 0.00 -> 81.4 mm, vias 0 -> 3
- net /+BATT_{SENSE}/ON: track 0.00 -> 66.6 mm, vias 0 -> 4
- net /BOOT: track 0.00 -> 62.1 mm, vias 0 -> 2
- net /D+: track 0.00 -> 58.2 mm
- net /D-: track 0.00 -> 56.7 mm
- net /BUTTON_{PWR}: track 0.00 -> 46.9 mm, vias 0 -> 2
- net GND: track 0.00 -> 43.3 mm, vias 0 -> 90
- net +5V: track 0.00 -> 32.4 mm, vias 0 -> 1
- net /IO2: track 0.00 -> 26.1 mm
- net /RX: track 0.00 -> 24.1 mm, vias 0 -> 2
- net /Power/+BATT_{switched}: track 0.00 -> 23.7 mm, vias 0 -> 1
- net Net-(D2-K): track 0.00 -> 22.5 mm, vias 0 -> 2
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Other:
- board text added: "JLCJLCJLCJLC"
