File: source/geheimbadge-controller/Battery.kicad_sch (KiCad schematic)
At the start: 9 parts, among them U1 XC5011

Commit message: finalized all designs
Parts:
- R2: value 1k -> 470; LCSC Part C21190 -> C23179
Other:
- note added: "I_{BAT} = V_{PROG}/R_{PROG} * 88 V_{PROG} = 1V I_{BAT} = 0.187A"
- note removed: "I_{BAT} = V_{PROG}/R_{PROG} * 1000 V_{PROG} = 1V I_{BAT} = 1A"
Changed lines of the file:
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@@
 		)
 	)
-	(text "I_{BAT} = V_{PROG}/R_{PROG} * 1000\nV_{PROG} = 1V\nI_{BAT} = 1A"
+	(text "I_{BAT} = V_{PROG}/R_{PROG} * 88\nV_{PROG} = 1V\nI_{BAT} = 0.187A"
 		(exclude_from_sim no)
 		(at 37.846 76.454 0)
@@
 					(unit 1)
 				)
-				(path "/5477044b-5ae5-4ed6-bb7d-f5f3cc95a2d4"
-					(reference "TP5")
-					(unit 1)
-				)
 			)
 		)
@@
 				(path "/5477044b-5ae5-4ed6-bb7d-f5f3cc95a2d4/3b6c4b5b-cb65-4de9-a343-7537d4c191c3/d6562b77-a863-48d7-8398-6af7a6dd4dde"
 					(reference "U1")
-					(unit 1)
-				)
-				(path "/5477044b-5ae5-4ed6-bb7d-f5f3cc95a2d4"
-					(reference "U2")
 					(unit 1)
 				)
@@
 					(unit 1)
 				)
-				(path "/5477044b-5ae5-4ed6-bb7d-f5f3cc95a2d4"
-					(reference "R12")
-					(unit 1)
-				)
 			)
 		)
@@
 					(unit 1)
 				)
-				(path "/5477044b-5ae5-4ed6-bb7d-f5f3cc95a2d4"
-					(reference "TP6")
-					(unit 1)
-				)
 			)
 		)
@@
 				(path "/5477044b-5ae5-4ed6-bb7d-f5f3cc95a2d4/3b6c4b5b-cb65-4de9-a343-7537d4c191c3/d6562b77-a863-48d7-8398-6af7a6dd4dde"
 					(reference "C1")
-					(unit 1)
-				)
-				(path "/5477044b-5ae5-4ed6-bb7d-f5f3cc95a2d4"
-					(reference "C2")
 					(unit 1)
 				)
@@
 			)
 		)
-		(property "Value" "1k"
+		(property "Value" "470"
 			(at 43.18 57.15 0)
 			(effects
@@
 			)
 		)
-		(property "LCSC Part" "C21190"
+		(property "LCSC Part" "C23179"
 			(at 45.72 55.88 0)
 			(effects
@@
 				(path "/5477044b-5ae5-4ed6-bb7d-f5f3cc95a2d4/3b6c4b5b-cb65-4de9-a343-7537d4c191c3/d6562b77-a863-48d7-8398-6af7a6dd4dde"
 					(reference "R2")
-					(unit 1)
-				)
-				(path "/5477044b-5ae5-4ed6-bb7d-f5f3cc95a2d4"
-					(reference "R13")
 					(unit 1)
 				)
@@
 					(unit 1)
 				)
-				(path "/5477044b-5ae5-4ed6-bb7d-f5f3cc95a2d4"
-					(reference "C3")
-					(unit 1)
-				)
