File: source/geheimbadge-controller/Power.kicad_sch (KiCad schematic)
At the start: 20 parts, among them U3 TLV62568DBVR, U4 XT1861B502SR-G

Commit message: finalized all designs
Parts:
- added D4, D5: 1N4148WS, Diode_SMD:D_SOD-323, symbol Diode:1N4148WS
- added Q7: AO3401A, Package_TO_SOT_SMD:SOT-23, symbol Transistor_FET:AO3401A
- added Q8: AO3400A, Package_TO_SOT_SMD:SOT-23, symbol Transistor_FET:AO3400A
- added R27, R28, R29: 10k, Resistor_SMD:R_0603_1608Metric, symbol Device:R
- L1, L2: value 2.2uH -> 10uH; footprint Inductor_SMD:L_1008_2520Metric -> Inductor_SMD:L_Chilisin_BMRx00060630; LCSC Part C3040393 -> C2827354
Connections:
- net +5V: now also Q7.2 (S), R27.2
- net +VDC: now also Q7.3 (D)
- net GND: now also Q8.2 (S), R28.1
- net VBUS: now also R29.2
- net at R22.2, TP15.1, U4.1 (CE): now also D5.1 (K)
- new net: D4.1 (K), Q7.1 (G), R27.1
- new net: D4.2 (A), D5.2 (A), Q8.3 (D)
- new net: Q8.1 (G), R28.2, R29.1
Other:
- moved on the sheet: C8, C9, L2, R22, TP14, TP15, U4
