File: source/geheimbadge-controller/SAO.kicad_sch (KiCad schematic)
At the start: 1 part, among them J3 SAOv2

Commit message: finalized all designs
Parts:
- J3: now left out of the parts list
Changed lines of the file:
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@@
 		(unit 1)
 		(exclude_from_sim no)
-		(in_bom yes)
+		(in_bom no)
 		(on_board yes)
 		(dnp yes)
@@
 					(unit 1)
 				)
-				(path "/5477044b-5ae5-4ed6-bb7d-f5f3cc95a2d4"
-					(reference "J1")
-					(unit 1)
-				)
